File: MC1496-Mixer.sch (KiCad schematic (older format))
At the start: 20 parts

Commit message: added image
Parts:
- added C?: .1uF, symbol Xenir:Capacitor
- added Q?: 2N3904, Package_TO_SOT_THT:TO-92_Inline, symbol Transistor_BJT:2N3904
- added R?: 1k, symbol Xenir:Resistor
Connections:
- net +12V: now also C?.2, Q?.3 (C)
- net GND: now also R?.2
- new net: Q?.1 (E), R?.1
- new net: C?.1, Q?.2 (B)
Other:
- note added: "Output\nSignal"
Changed lines of the file:
@@
 	6550 2300 6550 3000
 Wire Wire Line
-	6300 2850 6300 2300
-Wire Wire Line
 	6300 2300 6550 2300
 Connection ~ 6550 2300
@@
 Text Notes 3800 2000 0    50   ~ 0
 Modulation\nSignal
-Text Notes 4600 2000 0    50   ~ 0
+Text Notes 4650 2000 0    50   ~ 0
 Carrier\nInput
 $Comp
@@
 EndData
 $EndBitmap
+$Comp
+L Transistor_BJT:2N3904 Q?
+U 1 1 61F59F91
+P 7400 2750
+F 0 "Q?" H 7600 2825 50  0000 L CNN
+F 1 "2N3904" H 7600 2750 50  0000 L CNN
+F 2 "Package_TO_SOT_THT:TO-92_Inline" H 7600 2675 50  0001 L CIN
+F 3 "https://www.fairchildsemi.com/datasheets/2N/2N3904.pdf" H 7400 2750 50  0001 L CNN
+	1    7400 2750
+	1    0    0    -1
+$EndComp
+$Comp
+L Xenir:Resistor R?
+U 1 1 61F5AEFB
+P 7500 3350
+F 0 "R?" H 7500 3425 28  0000 C CNN
+F 1 "1k" H 7500 3275 28  0000 C CNN
+F 2 "" H 7500 3250 50  0001 C CNN
+F 3 "" H 7500 3250 50  0001 C CNN
+	1    7500 3350
+	0    1    1    0
+$EndComp
+Wire Wire Line
+	6750 2300 7500 2300
+Wire Wire Line
+	7500 2300 7500 2550
+Connection ~ 6750 2300
+$Comp
+L power:GND #PWR?
+U 1 1 61F5CFC9
+P 7500 3550
+F 0 "#PWR?" H 7500 3300 50  0001 C CNN
+F 1 "GND" H 7500 3400 50  0000 C CNN
+F 2 "" H 7500 3550 50  0001 C CNN
+F 3 "" H 7500 3550 50  0001 C CNN
+	1    7500 3550
+	1    0    0    -1
+$EndComp
+Wire Wire Line
+	6300 2300 6300 2750
+$Comp
+L Xenir:Capacitor C?
+U 1 1 61F5DC62
+P 7050 2750
+F 0 "C?" H 7050 2875 28  0000 C CNN
+F 1 ".1uF" H 7050 2625 28  0000 C CNN
+F 2 "" H 7050 2600 50  0001 C CNN
+F 3 "" H 7050 2600 50  0001 C CNN
+	1    7050 2750
+	-1   0    0    1
+$EndComp
+Wire Wire Line
+	6900 2750 6300 2750
+Connection ~ 6300 2750
+Wire Wire Line
+	6300 2750 6300 2850
+Wire Wire Line
+	7500 2950 7500 3050
+Wire Wire Line
+	7500 3050 7850 3050
+Connection ~ 7500 3050
+Wire Wire Line
+	7500 3050 7500 3150
+Text Notes 7900 3150 0    50   ~ 0
+Output\nSignal
 $EndSCHEMATC

Commit message: annot
Parts:
- gave numbers to parts that had none: 23
Changed lines of the file:
@@
 $EndDescr
 $Comp
-L Xenir:Resistor R?
+L Xenir:Resistor R9
 U 1 1 61F21B4D
 P 4700 4100
-F 0 "R?" H 4700 4175 28  0000 C CNN
+F 0 "R9" H 4700 4175 28  0000 C CNN
 F 1 "1k" H 4700 4025 28  0000 C CNN
 F 2 "" H 4700 4000 50  0001 C CNN
@@
 $EndComp
 $Comp
-L power:+12V #PWR?
+L power:+12V #PWR09
 U 1 1 61F22BB7
 P 6550 2300
-F 0 "#PWR?" H 6550 2150 50  0001 C CNN
+F 0 "#PWR09" H 6550 2150 50  0001 C CNN
 F 1 "+12V" H 6550 2440 50  0000 C CNN
 F 2 "" H 6550 2300 50  0001 C CNN
@@
 $EndComp
 $Comp
-L Xenir:Resistor R?
+L Xenir:Resistor R10
 U 1 1 61F23577
 P 6300 3050
-F 0 "R?" H 6300 3125 28  0000 C CNN
+F 0 "R10" H 6300 3125 28  0000 C CNN
 F 1 "3.3k" H 6300 2975 28  0000 C CNN
 F 2 "" H 6300 2950 50  0001 C CNN
@@
 $EndComp
 $Comp
-L Xenir:Resistor R?
+L Xenir:Resistor R11
 U 1 1 61F2429C
 P 6550 3200
-F 0 "R?" H 6550 3275 28  0000 C CNN
+F 0 "R11" H 6550 3275 28  0000 C CNN
 F 1 "3.3k" H 6550 3125 28  0000 C CNN
 F 2 "" H 6550 3100 50  0001 C CNN
@@
 Connection ~ 6550 2300
 $Comp
-L Xenir:Resistor R?
+L Xenir:Resistor R1
 U 1 1 61F27C75
 P 2750 3000
-F 0 "R?" H 2750 3075 28  0000 C CNN
+F 0 "R1" H 2750 3075 28  0000 C CNN
 F 1 "1k" H 2750 2925 28  0000 C CNN
 F 2 "" H 2750 2900 50  0001 C CNN
@@
 $EndComp
 $Comp
-L Xenir:MC1496 U?
+L Xenir:MC1496 U1
 U 1 1 61F29B1A
 P 5500 3150
-F 0 "U?" H 5450 3250 50  0000 C CNN
+F 0 "U1" H 5450 3250 50  0000 C CNN
 F 1 "MC1496" H 5500 3350 50  0000 C CNN
 F 2 "" H 5500 3350 50  0001 C CNN
@@
 	4900 3400 4300 3400
 $Comp
-L power:+12V #PWR?
+L power:+12V #PWR02
 U 1 1 61F2C31B
 P 2750 2450
-F 0 "#PWR?" H 2750 2300 50  0001 C CNN
+F 0 "#PWR02" H 2750 2300 50  0001 C CNN
 F 1 "+12V" H 2750 2590 50  0000 C CNN
 F 2 "" H 2750 2450 50  0001 C CNN
@@
 	2750 3200 2750 3400
 $Comp
-L Xenir:Resistor R?
+L Xenir:Resistor R8
 U 1 1 61F2CE90
 P 4500 3250
-F 0 "R?" H 4500 3325 28  0000 C CNN
+F 0 "R8" H 4500 3325 28  0000 C CNN
 F 1 "47" H 4500 3175 28  0000 C CNN
 F 2 "" H 4500 3150 50  0001 C CNN
@@
 	4500 4100 4500 4250
 $Comp
-L Xenir:BNC J?
+L Xenir:BNC J2
 U 1 1 61F2F8C6
 P 4750 2200
-F 0 "J?" H 4650 2050 50  0000 C CNN
+F 0 "J2" H 4650 2050 50  0000 C CNN
 F 1 "BNC" H 4750 2350 50  0000 C CNN
 F 2 "" H 4750 2350 50  0001 C CNN
@@
 $EndComp
 $Comp
-L power:GND #PWR?
+L power:GND #PWR07
 U 1 1 61F30922
 P 4550 2200
-F 0 "#PWR?" H 4550 1950 50  0001 C CNN
+F 0 "#PWR07" H 4550 1950 50  0001 C CNN
 F 1 "GND" H 4550 2050 50  0000 C CNN
 F 2 "" H 4550 2200 50  0001 C CNN
@@
 $EndComp
 $Comp
-L power:GND #PWR?
+L power:GND #PWR08
 U 1 1 61F31038
 P 6050 4250
-F 0 "#PWR?" H 6050 4000 50  0001 C CNN
+F 0 "#PWR08" H 6050 4000 50  0001 C CNN
 F 1 "GND" H 6050 4100 50  0000 C CNN
 F 2 "" H 6050 4250 50  0001 C CNN
@@
 	4750 2400 4750 2500
 $Comp
-L Xenir:Resistor R?
+L Xenir:Resistor R2
 U 1 1 61F347EC
 P 2750 3750
-F 0 "R?" H 2750 3825 28  0000 C CNN
+F 0 "R2" H 2750 3825 28  0000 C CNN
 F 1 "1k" H 2750 3675 28  0000 C CNN
 F 2 "" H 2750 3650 50  0001 C CNN
@@
 $EndComp
 $Comp
-L Xenir:Resistor R?
+L Xenir:Resistor R3
 U 1 1 61F34C9D
 P 2750 4550
-F 0 "R?" H 2750 4625 28  0000 C CNN
+F 0 "R3" H 2750 4625 28  0000 C CNN
 F 1 "1k" H 2750 4475 28  0000 C CNN
 F 2 "" H 2750 4450 50  0001 C CNN
@@
 $EndComp
 $Comp
-L Xenir:Capacitor C?
+L Xenir:Capacitor C1
 U 1 1 61F35D1E
 P 2400 3750
-F 0 "C?" H 2400 3875 28  0000 C CNN
+F 0 "C1" H 2400 3875 28  0000 C CNN
 F 1 ".1uF" H 2400 3625 28  0000 C CNN
 F 2 "" H 2400 3600 50  0001 C CNN
@@
 Connection ~ 2750 3400
 $Comp
-L power:GND #PWR?
+L power:GND #PWR01
 U 1 1 61F3698A
 P 2400 3900
-F 0 "#PWR?" H 2400 3650 50  0001 C CNN
+F 0 "#PWR01" H 2400 3650 50  0001 C CNN
 F 1 "GND" H 2400 3750 50  0000 C CNN
 F 2 "" H 2400 3900 50  0001 C CNN
@@
 	2750 3950 2750 4350
 $Comp
-L power:GND #PWR?
+L power:GND #PWR03
 U 1 1 61F3BD38
 P 2750 4750
-F 0 "#PWR?" H 2750 4500 50  0001 C CNN
+F 0 "#PWR03" H 2750 4500 50  0001 C CNN
 F 1 "GND" H 2750 4600 50  0000 C CNN
 F 2 "" H 2750 4750 50  0001 C CNN
@@
 $EndComp
 $Comp
-L Xenir:Resistor R?
+L Xenir:Resistor R4
 U 1 1 61F3E5C8
 P 3400 3700
-F 0 "R?" H 3400 3775 28  0000 C CNN
+F 0 "R4" H 3400 3775 28  0000 C CNN
 F 1 "100" H 3400 3625 28  0000 C CNN
 F 2 "" H 3400 3600 50  0001 C CNN
@@
 $EndComp
 $Comp
-L Xenir:Resistor R?
+L Xenir:Resistor R5
 U 1 1 61F3F0AA
 P 3400 3950
-F 0 "R?" H 3400 4025 28  0000 C CNN
+F 0 "R5" H 3400 4025 28  0000 C CNN
 F 1 "100" H 3400 3875 28  0000 C CNN
 F 2 "" H 3400 3850 50  0001 C CNN
@@
 Connection ~ 2750 3950
 $Comp
-L Xenir:Resistor R?
+L Xenir:Resistor R6
 U 1 1 61F42C96
 P 3600 4450
-F 0 "R?" H 3600 4525 28  0000 C CNN
+F 0 "R6" H 3600 4525 28  0000 C CNN
 F 1 "680" H 3600 4375 28  0000 C CNN
 F 2 "" H 3600 4350 50  0001 C CNN
@@
 $EndComp
 $Comp
-L Xenir:Resistor R?
+L Xenir:Resistor R7
 U 1 1 61F435BC
 P 4000 4450
-F 0 "R?" H 4000 4525 28  0000 C CNN
+F 0 "R7" H 4000 4525 28  0000 C CNN
 F 1 "680" H 4000 4375 28  0000 C CNN
 F 2 "" H 4000 4350 50  0001 C CNN
@@
 $EndComp
 $Comp
-L Xenir:Trimpot VR?
+L Xenir:Trimpot VR1
 U 1 1 61F43CD9
 P 3800 4700
-F 0 "VR?" H 3650 4400 50  0000 C CNN
+F 0 "VR1" H 3650 4400 50  0000 C CNN
 F 1 "Trimpot" H 3800 4800 50  0000 C CNN
 F 2 "" H 3650 4400 50  0001 C CNN
@@
 $EndComp
 $Comp
-L power:GND #PWR?
+L power:GND #PWR05
 U 1 1 61F45399
 P 3800 5050
-F 0 "#PWR?" H 3800 4800 50  0001 C CNN
+F 0 "#PWR05" H 3800 4800 50  0001 C CNN
 F 1 "GND" H 3800 4900 50  0000 C CNN
 F 2 "" H 3800 5050 50  0001 C CNN
@@
 	4500 4250 4900 4250
 $Comp
-L Xenir:Cap_Polarized C?
+L Xenir:Cap_Polarized C3
 U 1 1 61F4A2AE
 P 4350 4150
-F 0 "C?" H 4350 3925 28  0000 C CNN
+F 0 "C3" H 4350 3925 28  0000 C CNN
 F 1 "Cap_Polarized" H 4350 4200 28  0000 C CNN
 F 2 "" H 4350 4200 50  0001 C CNN
@@
 $EndComp
 $Comp
-L power:GND #PWR?
+L power:GND #PWR06
 U 1 1 61F4BD81
 P 4250 4300
-F 0 "#PWR?" H 4250 4050 50  0001 C CNN
+F 0 "#PWR06" H 4250 4050 50  0001 C CNN
 F 1 "GND" H 4250 4150 50  0000 C CNN
 F 2 "" H 4250 4300 50  0001 C CNN
@@
 	4250 3850 4900 3850
 $Comp
-L Xenir:BNC J?
+L Xenir:BNC J1
 U 1 1 61F4EF8E
 P 4000 2200
-F 0 "J?" H 3900 2050 50  0000 C CNN
+F 0 "J1" H 3900 2050 50  0000 C CNN
 F 1 "BNC" H 4000 2350 50  0000 C CNN
 F 2 "" H 4000 2350 50  0001 C CNN
@@
 $EndComp
 $Comp
-L power:GND #PWR?
+L power:GND #PWR04
 U 1 1 61F4EF98
 P 3800 2200
-F 0 "#PWR?" H 3800 1950 50  0001 C CNN
+F 0 "#PWR04" H 3800 1950 50  0001 C CNN
 F 1 "GND" H 3800 2050 50  0000 C CNN
 F 2 "" H 3800 2200 50  0001 C CNN
@@
 $EndComp
 $Comp
-L Xenir:Cap_Polarized C?
+L Xenir:Cap_Polarized C2
 U 1 1 61F4EFA2
 P 3900 2650
-F 0 "C?" H 3900 2425 28  0000 C CNN
+F 0 "C2" H 3900 2425 28  0000 C CNN
 F 1 "10uF" H 3900 2700 28  0000 C CNN
 F 2 "" H 3900 2700 50  0001 C CNN
@@
 	4700 3250 4750 3250
 $Comp
-L Xenir:Capacitor C?
+L Xenir:Capacitor C4
 U 1 1 61F53BE8
 P 4750 2650
-F 0 "C?" H 4750 2775 28  0000 C CNN
+F 0 "C4" H 4750 2775 28  0000 C CNN
 F 1 ".1uF" H 4750 2525 28  0000 C CNN
 F 2 "" H 4750 2500 50  0001 C CNN
@@
 Carrier\nInput
 $Comp
-L Xenir:Resistor R?
+L Xenir:Resistor R12
 U 1 1 61F55AD7
 P 6750 3500
-F 0 "R?" H 6750 3575 28  0000 C CNN
+F 0 "R12" H 6750 3575 28  0000 C CNN
 F 1 "10k" H 6750 3425 28  0000 C CNN
 F 2 "" H 6750 3400 50  0001 C CNN
@@
 Data
 89 50 4E 47 0D 0A 1A 0A 00 00 00 0D 49 48 44 52 00 00 04 B0 00 00 02 5A 08 02 00 00 00 B0 4C 29
-46 00 00 00 03 73 42 49 54 08 08 08 DB E1 4F E0 00 00 00 09 70 48 59 73 00 00 12 74 00 00 12 74
-01 DE 66 1F 78 00 00 20 00 49 44 41 54 78 9C EC DD 79 9C 5C 65 95 37 F0 DF 39 CF BD 55 D5 7B 67
+46 00 00 00 03 73 42 49 54 08 08 08 DB E1 4F E0 00 00 00 09 70 48 59 73 00 00 12 5C 00 00 12 5C
+01 68 C4 36 89 00 00 20 00 49 44 41 54 78 9C EC DD 79 9C 5C 65 95 37 F0 DF 39 CF BD 55 D5 7B 67
 5F 3A FB 4A 08 81 B0 64 81 C8 26 30 11 88 61 91 E0 82 F3 EA E8 A8 88 0B A2 02 02 3A 0A 3A CE A8
 8C 8C 2B 8E 08 88 28 A0 20 10 25 2C 06 90 2D 64 85 24 42 16 C8 4A C8 BE F7 5E 55 F7 3E CF 79 FF
@@
 $EndBitmap
 $Comp
-L Transistor_BJT:2N3904 Q?
+L Transistor_BJT:2N3904 Q1
 U 1 1 61F59F91
 P 7400 2750
-F 0 "Q?" H 7600 2825 50  0000 L CNN
+F 0 "Q1" H 7600 2825 50  0000 L CNN
 F 1 "2N3904" H 7600 2750 50  0000 L CNN
 F 2 "Package_TO_SOT_THT:TO-92_Inline" H 7600 2675 50  0001 L CIN
@@
 $EndComp
 $Comp
-L Xenir:Resistor R?
+L Xenir:Resistor R13
 U 1 1 61F5AEFB
 P 7500 3350
-F 0 "R?" H 7500 3425 28  0000 C CNN
+F 0 "R13" H 7500 3425 28  0000 C CNN
 F 1 "1k" H 7500 3275 28  0000 C CNN
 F 2 "" H 7500 3250 50  0001 C CNN
@@
 Connection ~ 6750 2300
 $Comp
-L power:GND #PWR?
+L power:GND #PWR010
 U 1 1 61F5CFC9
 P 7500 3550
-F 0 "#PWR?" H 7500 3300 50  0001 C CNN
+F 0 "#PWR010" H 7500 3300 50  0001 C CNN
 F 1 "GND" H 7500 3400 50  0000 C CNN
 F 2 "" H 7500 3550 50  0001 C CNN
@@
 	6300 2300 6300 2750
 $Comp
-L Xenir:Capacitor C?
+L Xenir:Capacitor C5
 U 1 1 61F5DC62
 P 7050 2750
-F 0 "C?" H 7050 2875 28  0000 C CNN
+F 0 "C5" H 7050 2875 28  0000 C CNN
 F 1 ".1uF" H 7050 2625 28  0000 C CNN
 F 2 "" H 7050 2600 50  0001 C CNN

Commit message: removed output cap
Parts:
- removed C5: .1uF, symbol Xenir:Capacitor
- VR1: value Trimpot -> 50k
Connections:
- net +12V: now also Q1.2 (B)
Other:
- note added: "Page 8 - https://www.onsemi.com/pdf/datasheet/mc1496-d.pdf"
- note added: "Resistor Divider Biasing"
- note removed: "Carrier Adjust\n(DSBSC <-> AM)"
- moved on the sheet: C1, C2, C3, C4, J1, J2, Q1, R1, R10, R11, R12, R13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

Commit message: fixes
Parts:
- C3: value Cap_Polarized -> 470uF
Other:
- note added: "Carrier\nAdjust"
Changed lines of the file:
@@
 P 3850 3750
 F 0 "C3" H 3850 3525 28  0000 C CNN
-F 1 "Cap_Polarized" H 3850 3800 28  0000 C CNN
+F 1 "470uF" H 3850 3800 28  0000 C CNN
 F 2 "" H 3850 3800 50  0001 C CNN
 F 3 "" H 3850 3800 50  0001 C CNN
@@
 Wire Wire Line
 	5800 2350 6700 2350
+Text Notes 3700 4650 2    50   ~ 0
+Carrier\nAdjust
 $EndSCHEMATC

Commit message: gg
Other:
- note added: "Carrier\nInput\n300mV p-p"
- note added: "Modulation\nSignal\n300mV p-p"
- note removed: "Carrier\nInput"
- note removed: "Modulation\nSignal"
Changed lines of the file:
@@
 Resistor Divider Biasing
 Text Notes 3300 1600 0    50   ~ 0
-Modulation\nSignal
+Modulation\nSignal\n300mV p-p
 Text Notes 4150 1600 0    50   ~ 0
-Carrier\nInput
+Carrier\nInput\n300mV p-p
 $Comp
 L Xenir:Resistor R12
